Commit message: Rebuilding pioneer model.

File: p3at/urdf/p3at.xacro (robot description, xacro)
@@ -2,5 +2,74 @@
 <robot xmlns:xacro="http://ros.org/wiki/xacro" name="p3at">
 <!-- Macros -->
-	<xacro:macro name="p3at_wheel" params="fb lr">
+	<xacro:macro name="p3at_wheel" params="fb lr xyz reflect">
+		<!-- Axle -->
+		<link name="p3at_${fb}_${lr}_axle">
+			<inertial>
+				<mass value="0.1"/>
+				<origin xyz="0 0 0"/>
+				<inertia ixx="1.0" ixy="0.0" ixz="0.0"
+					 iyy="1.0" iyz="0.0" izz="1.0"/>
+	  	 	</inertial>
+			<visual name="base_visual">
+				<origin xyz="0 0 0" rpy="0 0 0"/>
+				<geometry name="pioneer_geom">
+					<mesh filename="package://p2os_urdf/meshes/p3at_meshes/axle.stl"/>
+				</geometry>
+				<material name="AxleGrey">
+					<color rgba="0.5 0.5 0.5 1"/>
+				</material>
+			</visual>
+			<collision>
+				<origin xyz="0 0 0" rpy="0 0 0"/>
+				<geometry>
+					<box size="0 0 0"/>
+				</geometry>
+			</collision>
+		</link>
+		<gazebo reference="p3at_${fb}_${lr}_axle">
+			<material value="Gazebo/Grey"/>
+		</gazebo>
+		<joint name="base_${fb}_${lr}_axle_joint" type="continuous">
+			<origin xyz="${xyz}" rpy="0 0 0"/>
+			<parent link="base_link"/>
+			<child link="p3at_${fb}_${lr}_axle"/>
+			<axis xyz="0 1 0"/>
+			<anchor xyz="0 0 0"/>
+			<limit effort="100" velocity="100" />
+			<joint_properties damping="0.7"/>
+		</joint>
+		<!-- Wheel-Hub -->
+		<link name="p3at_${fb}_${lr}_hub">
+			<inertial>
+				<mass value="0.1"/>
+				<origin xyz="0 0 0"/>
+				<inertia ixx="1.0" ixy="0.0" ixz="0.0"
+					 iyy="1.0" iyz="0.0" izz="1.0"/>
+	  	 	</inertial>
+			<visual name="base_visual">
+				<origin xyz="0 0 0" rpy="0 0 0"/>
+				<geometry name="pioneer_geom">
+					<mesh filename="package://p2os_urdf/meshes/p3at_meshes/${lr}_hubcap.stl"/>
+				</geometry>
+				<material name="HubcapYellow">
+					<color rgba="1.0 0.811 0.151 1.0"/>
+				</material>
+			</visual>
+			<collision>
+				<origin xyz="0 0 0" rpy="0 0 0"/>
+				<geometry>
+					<box size="0 0 0"/>
+				</geometry>
+			</collision>
+		</link>
+		<gazebo reference="p3at_${fb}_${lr}_hub">
+			<material value="Gazebo/Yellow"/>
+		</gazebo>
+		<joint name="base_${fb}_${lr}_hub_joint" type="fixed">
+			<origin xyz="0 ${reflect*0.041} 0" rpy="0 0 0"/>
+			<parent link="p3at_${fb}_${lr}_axle"/>
+			<child link="p3at_${fb}_${lr}_hub"/>
+		</joint>
+		<!-- Wheel -->
 		<link name="p3at_${fb}_${lr}_wheel">
 			<inertial>
@@ -25,4 +94,5 @@
 			</collision>
 		</link>
+<!--
 		<joint name="p3at_${fb}_${lr}_wheel_joint" type="continuous">
 			<axis xyz="0 1 0"/>
@@ -31,6 +101,12 @@
 			<joint_properties damping="0.7"/>
 			<origin xyz="0 0 0" rpy="0 0 0"/>
-			<parent link="p3at_front_${suffix}_hub"/>
-			<child link="p3at_front_${suffix}_wheel"/>
+			<parent link="p3at_${fb}_${lr}_hub"/>
+			<child link="p3at_${fb}_${lr}_wheel"/>
+		</joint>
+-->
+		<joint name="p3at_${fb}_${lr}_wheel_joint" type="fixed">
+			<origin xyz="0 0 0" rpy="0 0 0"/>
+			<parent link="p3at_${fb}_${lr}_hub"/>
+			<child link="p3at_${fb}_${lr}_wheel"/>
 		</joint>
 		<gazebo reference="p3at_${fb}_${lr}_wheel">
@@ -44,8 +120,9 @@
 		</gazebo>
 	</xacro:macro>
-<!-- Chassis -->
+<!-- Robot definition -->
+	<!-- Chassis -->
 	<link name="base_link">
 		<inertial>
-			<mass value="10.0"/>
+			<mass value="100.0"/>
 			<origin xyz="0 0 0.177"/>
 			<inertia ixx="0.3338" ixy="0.0" ixz="0.0"
@@ -105,149 +182,27 @@
 		<material value="Gazebo/Black"/>
 	</gazebo>
-<!-- Front Axles + Wheels + Hubcaps -->
-<xacro:macro name="p3at_front" params="suffix reflect">
-	<link name="p3at_front_${suffix}_axle">
-		<inertial>
-			<mass value="0.1"/>
-			<origin xyz="0 0 0"/>
-			<inertia ixx="1.0" ixy="0.0" ixz="0.0"
-				 iyy="1.0" iyz="0.0" izz="1.0"/>
-  	 	</inertial>
-	<visual name="base_visual">
-		<origin xyz="0 0 0" rpy="0 0 0"/>
-		<geometry name="pioneer_geom">
-			<mesh filename="package://p2os_urdf/meshes/p3at_meshes/axle.stl"/>
-		</geometry>
-		<material name="AxleGrey">
-			<color rgba="0.5 0.5 0.5 1"/>
-		</material>
-	</visual>
-	<collision>
-		<origin xyz="0 0 0" rpy="0 0 0"/>
-		<geometry>
-			<box size="0 0 0"/>
-		</geometry>
-	</collision>
-	</link>
-	<gazebo reference="p3at_front_${suffix}_axle">
-		<material value="Gazebo/Grey"/>
+	<xacro:p3at_wheel lr="left" fb="front"  xyz=" 0.135 0.156 0.111" reflect="1" />
+	<xacro:p3at_wheel lr="left" fb="back"   xyz="-0.135 0.156 0.111" reflect="1" />
+	<xacro:p3at_wheel lr="right" fb="front" xyz=" 0.135 -0.156 0.111" reflect="-1" />
+	<xacro:p3at_wheel lr="right" fb="back"  xyz="-0.135 -0.156 0.111" reflect="-1" />
+<xacro:macro name="p3at_controller" params="ns">
+	<gazebo>
+		<plugin name="skid_steer_drive_controller" filename="libgazebo_ros_skid_steer_drive.so">
+			<updateRate>100.0</updateRate>
+			<robotNamespace>${ns}</robotNamespace>
+			<leftFrontJoint>base_front_left_axle_joint</leftFrontJoint>
+			<rightFrontJoint>base_front_right_axle_joint</rightFrontJoint>
+			<leftRearJoint>base_back_left_axle_joint</leftRearJoint>
+			<rightRearJoint>base_back_right_axle_joint</rightRearJoint>
+			<wheelSeparation>0.4</wheelSeparation>
+			<wheelDiameter>0.215</wheelDiameter>
+			<robotBaseFrame>base_link</robotBaseFrame>
+			<odometryFrame>odom</odometryFrame>
+			<torque>200</torque>
+			<commandTopic>cmd_vel</commandTopic>
+			<odometryTopic>odom</odometryTopic>
+			<broadcastTF>1</broadcastTF>
+		</plugin>
 	</gazebo>
-	<joint name="base_front_${suffix}_axle_joint" type="fixed">
-		<origin xyz="0.135 ${reflect*0.156} 0.111" rpy="0 0 0"/>
-		<parent link="base_link"/>
-		<child link="p3at_front_${suffix}_axle"/>
-	</joint>
-	<link name="p3at_front_${suffix}_hub">
-		<inertial>
-			<mass value="0.1"/>
-			<origin xyz="0 0 0"/>
-			<inertia ixx="1.0" ixy="0.0" ixz="0.0"
-				 iyy="1.0" iyz="0.0" izz="1.0"/>
-  	 	</inertial>
-	<visual name="base_visual">
-		<origin xyz="0 0 0" rpy="0 0 0"/>
-		<geometry name="pioneer_geom">
-			<mesh filename="package://p2os_urdf/meshes/p3at_meshes/${suffix}_hubcap.stl"/>
-		</geometry>
-		<material name="HubcapYellow">
-			<color rgba="1.0 0.811 0.151 1.0"/>
-		</material>
-	</visual>
-	<collision>
-		<origin xyz="0 0 0" rpy="0 0 0"/>
-		<geometry>
-			<box size="0 0 0"/>
-		</geometry>
-	</collision>
-	</link>
-	<gazebo reference="p3at_front_${suffix}_hub">
-		<material value="Gazebo/Yellow"/>
-	</gazebo>
-	<joint name="base_front_${suffix}_hub_joint" type="fixed">
-		<origin xyz="0 ${reflect*0.041} 0" rpy="0 0 0"/>
-		<parent link="p3at_front_${suffix}_axle"/>
-		<child link="p3at_front_${suffix}_hub"/>
-	</joint>
-<!-- Back Axles + Wheels + Hubcaps -->
-	<link name="p3at_back_${suffix}_axle">
-		<inertial>
-			<mass value="0.1"/>
-			<origin xyz="0 0 0"/>
-			<inertia ixx="1.0" ixy="0.0" ixz="0.0"
-				 iyy="1.0" iyz="0.0" izz="1.0"/>
-  	 	</inertial>
-	<visual name="base_visual">
-		<origin xyz="0 0 0" rpy="0 0 0"/>
-		<geometry name="pioneer_geom">
-			<mesh filename="package://p2os_urdf/meshes/p3at_meshes/axle.stl"/>
-		</geometry>
-		<material name="AxleGrey">
-			<color rgba="0.5 0.5 0.5 1"/>
-		</material>
-	</visual>
-	<collision>
-		<origin xyz="0 0 0" rpy="0 0 0"/>
-		<geometry>
-			<mesh filename="package://p2os_urdf/meshes/p3at_meshes/axle.stl"/>
-		</geometry>
-	</collision>
-	</link>
-	<gazebo reference="p3at_back_${suffix}_axle">
-		<material value="Gazebo/Grey"/>
-	</gazebo>
-	<joint name="bp3at_back_${suffix}_axle_joint" type="fixed">
-		<origin xyz="-0.134 ${reflect*0.156} 0.111" rpy="0 0 0"/>
-		<parent link="base_link"/>
-		<child link="p3at_back_${suffix}_axle"/>
-	</joint>
-	<link name="p3at_back_${suffix}_hub">
-		<inertial>
-			<mass value="0.1"/>
-			<origin xyz="0 0 0"/>
-			<inertia ixx="1.0" ixy="0.0" ixz="0.0"
-				 iyy="1.0" iyz="0.0" izz="1.0"/>
-  	 	</inertial>
-	<visual name="base_visual">
-		<origin xyz="0 0 0" rpy="0 0 0"/>
-		<geometry name="pioneer_geom">
-			<mesh filename="package://p2os_urdf/meshes/p3at_meshes/${suffix}_hubcap.stl"/>
-		</geometry>
-		<material name="HubcapYellow"/>
-	</visual>
-	<collision>
-		<origin xyz="0 0 0" rpy="0 0 0"/>
-		<geometry>
-			<mesh filename="package://p2os_urdf/meshes/p3at_meshes/${suffix}_hubcap.stl"/>
-		</geometry>
-	</collision>
-	</link>
-	<gazebo reference="p3at_back_${suffix}_hub">
-		<material value="Gazebo/Yellow"/>
-	</gazebo>
-	<joint name="p3at_back_${suffix}_hub_joint" type="fixed">
-		<origin xyz="-0 ${reflect*0.041} 0" rpy="0 0 0"/>
-		<parent link="p3at_back_${suffix}_axle"/>
-		<child link="p3at_back_${suffix}_hub"/>
-	</joint>
-</xacro:macro>
-<xacro:macro name="p3at_gazebo_ext" params="ns">
-<gazebo>
-  <plugin name="skid_steer_drive_controller" filename="libgazebo_ros_skid_steer_drive.so">
-    <updateRate>100.0</updateRate>
-    <robotNamespace>${ns}</robotNamespace>
-    <leftFrontJoint>p3at_front_left_wheel_joint</leftFrontJoint>
-    <rightFrontJoint>p3at_front_right_wheel_joint</rightFrontJoint>
-    <leftRearJoint>p3at_back_left_wheel_joint</leftRearJoint>
-    <rightRearJoint>p3at_back_right_wheel_joint</rightRearJoint>
-    <wheelSeparation>0.4</wheelSeparation>
-    <wheelDiameter>0.215</wheelDiameter>
-    <robotBaseFrame>base_link</robotBaseFrame>
-    <odometryFrame>odom</odometryFrame>
-    <torque>200</torque>
-    <commandTopic>cmd_vel</commandTopic>
-    <odometryTopic>odom</odometryTopic>
-    <broadcastTF>1</broadcastTF>
-  </plugin>
-</gazebo>
 </xacro:macro>
 </robot>

File: scout/urdf/scout.xacro (robot description, xacro)
@@ -2,4 +2,5 @@
 <robot xmlns:xacro="http://ros.org/wiki/xacro" name="scout">
 	<include filename="$(find p3at)/urdf/p3at.xacro"/>
+	<xacro:p3at_controller ns="scout" />
 <!--
 	<include filename="$(find sensors)/urdf/hokuyo.xacro"/>

Commit message: Made wheel joint continuous again.

File: p3at/urdf/p3at.xacro (robot description, xacro)
@@ -30,13 +30,4 @@
 			<material value="Gazebo/Grey"/>
 		</gazebo>
-		<joint name="base_${fb}_${lr}_axle_joint" type="continuous">
-			<origin xyz="${xyz}" rpy="0 0 0"/>
-			<parent link="base_link"/>
-			<child link="p3at_${fb}_${lr}_axle"/>
-			<axis xyz="0 1 0"/>
-			<anchor xyz="0 0 0"/>
-			<limit effort="100" velocity="100" />
-			<joint_properties damping="0.7"/>
-		</joint>
 		<!-- Wheel-Hub -->
 		<link name="p3at_${fb}_${lr}_hub">
@@ -66,9 +57,4 @@
 			<material value="Gazebo/Yellow"/>
 		</gazebo>
-		<joint name="base_${fb}_${lr}_hub_joint" type="fixed">
-			<origin xyz="0 ${reflect*0.041} 0" rpy="0 0 0"/>
-			<parent link="p3at_${fb}_${lr}_axle"/>
-			<child link="p3at_${fb}_${lr}_hub"/>
-		</joint>
 		<!-- Wheel -->
 		<link name="p3at_${fb}_${lr}_wheel">
@@ -94,16 +80,20 @@
 			</collision>
 		</link>
-<!--
-		<joint name="p3at_${fb}_${lr}_wheel_joint" type="continuous">
+		<!-- Wheel joints -->
+		<joint name="p3at_${fb}_${lr}_base_axle_joint" type="fixed">
+			<origin xyz="${xyz}" rpy="0 0 0"/>
+			<parent link="base_link"/>
+			<child link="p3at_${fb}_${lr}_axle"/>
+		</joint>
+		<joint name="p3at_${fb}_${lr}_axle_hub_joint" type="fixed">
+			<origin xyz="0 ${reflect*0.041} 0" rpy="0 0 0"/>
+			<parent link="p3at_${fb}_${lr}_axle"/>
+			<child link="p3at_${fb}_${lr}_hub"/>
+		</joint>
+		<joint name="p3at_${fb}_${lr}_hub_wheel_joint" type="continuous">
 			<axis xyz="0 1 0"/>
 			<anchor xyz="0 0 0"/>
 			<limit effort="100" velocity="100" />
 			<joint_properties damping="0.7"/>
-			<origin xyz="0 0 0" rpy="0 0 0"/>
-			<parent link="p3at_${fb}_${lr}_hub"/>
-			<child link="p3at_${fb}_${lr}_wheel"/>
-		</joint>
--->
-		<joint name="p3at_${fb}_${lr}_wheel_joint" type="fixed">
 			<origin xyz="0 0 0" rpy="0 0 0"/>
 			<parent link="p3at_${fb}_${lr}_hub"/>
@@ -120,9 +110,29 @@
 		</gazebo>
 	</xacro:macro>
+	<xacro:macro name="p3at_controller" params="ns">
+		<gazebo>
+			<plugin name="skid_steer_drive_controller" filename="libgazebo_ros_skid_steer_drive.so">
+				<updateRate>100.0</updateRate>
+				<robotNamespace>${ns}</robotNamespace>
+				<leftFrontJoint>p3at_front_left_hub_wheel_joint</leftFrontJoint>
+				<rightFrontJoint>p3at_front_right_hub_wheel_joint</rightFrontJoint>
+				<leftRearJoint>p3at_back_left_hub_wheel_joint</leftRearJoint>
+				<rightRearJoint>p3at_back_right_hub_wheel_joint</rightRearJoint>
+				<wheelSeparation>0.4</wheelSeparation>
+				<wheelDiameter>0.215</wheelDiameter>
+				<robotBaseFrame>base_link</robotBaseFrame>
+				<odometryFrame>odom</odometryFrame>
+				<torque>200</torque>
+				<commandTopic>cmd_vel</commandTopic>
+				<odometryTopic>odom</odometryTopic>
+				<broadcastTF>1</broadcastTF>
+			</plugin>
+		</gazebo>
+	</xacro:macro>
 <!-- Robot definition -->
 	<!-- Chassis -->
 	<link name="base_link">
 		<inertial>
-			<mass value="100.0"/>
+			<mass value="10.0"/>
 			<origin xyz="0 0 0.177"/>
 			<inertia ixx="0.3338" ixy="0.0" ixz="0.0"
@@ -149,5 +159,5 @@
 		<material value="Gazebo/Red"/>
 	</gazebo>
-<!-- Top -->
+	<!-- Top plate -->
 	<link name="top_plate">
 		<inertial>
@@ -186,23 +196,3 @@
 	<xacro:p3at_wheel lr="right" fb="front" xyz=" 0.135 -0.156 0.111" reflect="-1" />
 	<xacro:p3at_wheel lr="right" fb="back"  xyz="-0.135 -0.156 0.111" reflect="-1" />
-<xacro:macro name="p3at_controller" params="ns">
-	<gazebo>
-		<plugin name="skid_steer_drive_controller" filename="libgazebo_ros_skid_steer_drive.so">
-			<updateRate>100.0</updateRate>
-			<robotNamespace>${ns}</robotNamespace>
-			<leftFrontJoint>base_front_left_axle_joint</leftFrontJoint>
-			<rightFrontJoint>base_front_right_axle_joint</rightFrontJoint>
-			<leftRearJoint>base_back_left_axle_joint</leftRearJoint>
-			<rightRearJoint>base_back_right_axle_joint</rightRearJoint>
-			<wheelSeparation>0.4</wheelSeparation>
-			<wheelDiameter>0.215</wheelDiameter>
-			<robotBaseFrame>base_link</robotBaseFrame>
-			<odometryFrame>odom</odometryFrame>
-			<torque>200</torque>
-			<commandTopic>cmd_vel</commandTopic>
-			<odometryTopic>odom</odometryTopic>
-			<broadcastTF>1</broadcastTF>
-		</plugin>
-	</gazebo>
-</xacro:macro>
 </robot>

Commit message: Changed p3at params.

File: p3at/urdf/p3at.xacro (robot description, xacro)
@@ -106,6 +106,6 @@
 			<kd>1.0</kd>
 			<fdir1 value="1 0 0"/>
-			<mu1>1.0</mu1>
-			<mu2>1.0</mu2>
+			<mu1>0.6</mu1>
+			<mu2>0.2</mu2>
 		</gazebo>
 	</xacro:macro>
@@ -134,5 +134,5 @@
 	<link name="base_link">
 		<inertial>
-			<mass value="10.0"/>
+			<mass value="30.0"/>
 			<origin xyz="0 0 0.177"/>
 			<inertia ixx="0.3338" ixy="0.0" ixz="0.0"
